Commit message: Another new moveit config and urdf updates

File: rover_description/urdf/rover.urdf.xacro (robot description, xacro)
@@ -308,5 +308,5 @@
       upper="2.3562"
       velocity="0.25"
-      effort="0.0"
+      effort="120.0"
       />
   </joint>
@@ -365,5 +365,5 @@
       upper="1.0472"
       velocity="0.25"
-      effort="0.0"
+      effort="400.0"
       />
   </joint>
@@ -422,5 +422,5 @@
       upper="2.3562"
       velocity="0.5"
-      effort="0.0"
+      effort="100.0"
       /> <!-- really vel should be 1.2 -->
   </joint>
@@ -479,5 +479,5 @@
       upper="3.1416"
       velocity="0.5"
-      effort="0.0"
+      effort="25.0"
       /> <!-- really vel should be 1.2 -->
   </joint>
@@ -536,5 +536,5 @@
       upper="1.5708"
       velocity="0.5"
-      effort="0.0"
+      effort="25.0"
       /> <!-- really vel should be 1.2 -->
   </joint>
@@ -593,6 +593,12 @@
       upper="3.1416"
       velocity="0.5"
-      effort="0.0"
+      effort="25.0"
       /> <!-- really vel should be 1.2 -->
+  </joint>
+  <link name="tcp_link" />
+  <joint name="gripper_to_tcp" type="fixed">
+    <parent link="Arm_Gripper"/>
+    <child link="tcp_link"/>
+    <origin xyz="0 0.3 0" rpy="0 0 0"/>
   </joint>
   <xacro:rover_ros2_control use_gazebo="$(arg use_gazebo)"/>
