Commit message: Prepare for new EPOS-based gripper

File: rover_description/urdf/rover.control.xacro (robot description, xacro)
@@ -93,4 +93,12 @@
         <param name="differential_index">1</param>
       </joint>
+      <joint name="Arm_Gripper_Clamp">
+        <state_interface name="position"/>
+        <state_interface name="velocity"/>
+        <command_interface name="position"/>
+        <!-- <command_interface name="velocity"/> -->
+        <param name="epos_node_id">6</param>
+        <param name="position_target_scale">117000.0</param>
+      </joint>
     </ros2_control>
     <ros2_control name="RoverArmSteppers" type="system">

File: rover_description/urdf/rover.urdf.xacro (robot description, xacro)
@@ -601,4 +601,11 @@
     <child link="tcp_link"/>
     <origin xyz="0 0.3 0" rpy="0 0 0"/>
+  </joint>
+  <link name="dummy_gripper_link" />
+  <joint name="Arm_Gripper_Clamp" type="continuous">
+    <parent link="tcp_link" />
+    <child link="dummy_gripper_link" />
+    <origin xyz="0 0 0" rpy="0 0 0" />
+    <axis xyz="1 0 0" />
   </joint>
   <xacro:rover_ros2_control use_gazebo="$(arg use_gazebo)"/>
